File: docs/eagle/cap_meter.sch (EAGLE design)
At the start: 8 parts

Commit message: version 2.0
Parts:
- added PUSH_BUTTON_S3: MOMENTARY-SWITCH-SPST-PTH-6.0MM-KIT, SparkFun-Switches:MOMENTARY-SWITCH-SPST-PTH-6.0MM-KIT
- added R3: 10k, eagle-ltspice:RR1210
- added R4: 3.3K, eagle-ltspice:RR1210
- added R5: 1.8K, eagle-ltspice:RR1210
- added TEST_3_J3: ED555/2DS, DC_LOAD_AU:ED555/2DS
Connections:
- new net N$10: PUSH_BUTTON_S3.1, U$1.D10
- new net N$11: R3.2, U$1.D2
- new net N$12: R3.1, TEST_3_J3.1, U$1.D6
- new net N$13: R4.2, R5.1, U$1.D7
- net GND: now also PUSH_BUTTON_S3.2, R5.2, TEST_3_J3.2
- net VCC: now also R4.1, U$1.5.5V

Commit message: version 2.1-2
Parts:
- OLED: value (none) -> SSD1306
- R4: value 3.3K -> 1.8K
- R5: value 1.8K -> 3.1K
Other:
- moved on the sheet: PUSH_BUTTON_S2
Changed lines of the file:
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@@
 </classes>
 <parts>
-<part name="OLED" library="SparkFun-Connectors" library_urn="urn:adsk.eagle:library:513" deviceset="I2C_STANDARD" device="" package3d_urn="urn:adsk.eagle:package:38085/1"/>
+<part name="OLED" library="SparkFun-Connectors" library_urn="urn:adsk.eagle:library:513" deviceset="I2C_STANDARD" device="" package3d_urn="urn:adsk.eagle:package:38085/1" value="SSD1306"/>
 <part name="PUSH_BUTTON_S1" library="SparkFun-Switches" library_urn="urn:adsk.eagle:library:535" deviceset="MOMENTARY-SWITCH-SPST" device="-PTH-6.0MM-KIT" package3d_urn="urn:adsk.eagle:package:40170/1" value=""/>
 <part name="PUSH_BUTTON_S2" library="SparkFun-Switches" library_urn="urn:adsk.eagle:library:535" deviceset="MOMENTARY-SWITCH-SPST" device="-PTH-6.0MM-KIT" package3d_urn="urn:adsk.eagle:package:40170/1" value=""/>
@@
 <part name="SUPPLY5" library="supply2" library_urn="urn:adsk.eagle:library:372" deviceset="GND" device=""/>
 <part name="R3" library="eagle-ltspice" library_urn="urn:adsk.eagle:library:217" deviceset="R" device="R1210" package3d_urn="urn:adsk.eagle:package:13299/1" value="10k"/>
-<part name="R4" library="eagle-ltspice" library_urn="urn:adsk.eagle:library:217" deviceset="R" device="R1210" package3d_urn="urn:adsk.eagle:package:13299/1" value="3.3K"/>
-<part name="R5" library="eagle-ltspice" library_urn="urn:adsk.eagle:library:217" deviceset="R" device="R1210" package3d_urn="urn:adsk.eagle:package:13299/1" value="1.8K"/>
+<part name="R4" library="eagle-ltspice" library_urn="urn:adsk.eagle:library:217" deviceset="R" device="R1210" package3d_urn="urn:adsk.eagle:package:13299/1" value="1.8K"/>
+<part name="R5" library="eagle-ltspice" library_urn="urn:adsk.eagle:library:217" deviceset="R" device="R1210" package3d_urn="urn:adsk.eagle:package:13299/1" value="3.1K"/>
 <part name="SUPPLY6" library="supply2" library_urn="urn:adsk.eagle:library:372" deviceset="GND" device=""/>
 <part name="P+2" library="supply1" library_urn="urn:adsk.eagle:library:371" deviceset="VCC" device=""/>
@@
 <attribute name="VALUE" x="129.54" y="70.612" size="1.778" layer="96" font="vector" align="top-center"/>
 </instance>
-<instance part="PUSH_BUTTON_S2" gate="G$1" x="127" y="83.82" smashed="yes">
-<attribute name="NAME" x="127" y="85.344" size="1.778" layer="95" font="vector" align="bottom-center"/>
-<attribute name="VALUE" x="127" y="83.312" size="1.778" layer="96" font="vector" align="top-center"/>
+<instance part="PUSH_BUTTON_S2" gate="G$1" x="129.54" y="83.82" smashed="yes">
+<attribute name="NAME" x="129.54" y="85.344" size="1.778" layer="95" font="vector" align="bottom-center"/>
+<attribute name="VALUE" x="129.54" y="83.312" size="1.778" layer="96" font="vector" align="top-center"/>
 </instance>
 <instance part="R1" gate="G$1" x="71.12" y="35.56" smashed="yes" rot="R180">
@@
 </instance>
 <instance part="U$1" gate="G$1" x="101.6" y="78.74" smashed="yes"/>
-<instance part="P+1" gate="VCC" x="12.7" y="55.88" smashed="yes" rot="R180">
-<attribute name="VALUE" x="15.24" y="58.42" size="1.778" layer="96" rot="R270"/>
+<instance part="P+1" gate="VCC" x="12.7" y="43.18" smashed="yes" rot="R180">
+<attribute name="VALUE" x="15.24" y="45.72" size="1.778" layer="96" rot="R270"/>
 </instance>
 <instance part="SUPPLY1" gate="GND" x="7.62" y="45.72" smashed="yes">
@@
 <segment>
 <pinref part="P+1" gate="VCC" pin="VCC"/>
-<wire x1="12.7" y1="58.42" x2="12.7" y2="71.12" width="0.1524" layer="91"/>
+<wire x1="12.7" y1="45.72" x2="12.7" y2="71.12" width="0.1524" layer="91"/>
 <pinref part="OLED" gate="G$1" pin="2"/>
 <wire x1="12.7" y1="71.12" x2="5.08" y2="71.12" width="0.1524" layer="91"/>
@@
 <segment>
 <pinref part="PUSH_BUTTON_S2" gate="G$1" pin="2"/>
-<wire x1="132.08" y1="83.82" x2="144.78" y2="83.82" width="0.1524" layer="91"/>
+<wire x1="134.62" y1="83.82" x2="144.78" y2="83.82" width="0.1524" layer="91"/>
 <wire x1="144.78" y1="68.58" x2="144.78" y2="71.12" width="0.1524" layer="91"/>
 <pinref part="SUPPLY2" gate="GND" pin="GND"/>
 <pinref part="PUSH_BUTTON_S1" gate="G$1" pin="2"/>
-<wire x1="144.78" y1="71.12" x2="144.78" y2="81.28" width="0.1524" layer="91"/>
-<wire x1="144.78" y1="81.28" x2="144.78" y2="83.82" width="0.1524" layer="91"/>
+<wire x1="144.78" y1="71.12" x2="144.78" y2="83.82" width="0.1524" layer="91"/>
 <wire x1="134.62" y1="71.12" x2="144.78" y2="71.12" width="0.1524" layer="91"/>
 <junction x="144.78" y="71.12"/>
@@
 <pinref part="PUSH_BUTTON_S2" gate="G$1" pin="1"/>
 <pinref part="U$1" gate="G$1" pin="D8"/>
-<wire x1="121.92" y1="83.82" x2="111.76" y2="83.82" width="0.1524" layer="91"/>
+<wire x1="124.46" y1="83.82" x2="111.76" y2="83.82" width="0.1524" layer="91"/>
 </segment>
 </net>
@@
 </segment>
 </net>
-<net name="N$9" class="0">
-<segment>
-<pinref part="U$1" gate="G$1" pin="D12"/>
-<wire x1="119.38" y1="93.98" x2="111.76" y2="93.98" width="0.1524" layer="91"/>
-<wire x1="119.38" y1="99.06" x2="119.38" y2="93.98" width="0.1524" layer="91"/>
-<wire x1="119.38" y1="101.6" x2="119.38" y2="99.06" width="0.1524" layer="91"/>
-<wire x1="68.58" y1="101.6" x2="119.38" y2="101.6" width="0.1524" layer="91"/>
-<wire x1="66.04" y1="101.6" x2="68.58" y2="101.6" width="0.1524" layer="91"/>
-<wire x1="63.5" y1="101.6" x2="63.5" y2="35.56" width="0.1524" layer="91"/>
-<wire x1="66.04" y1="101.6" x2="63.5" y2="101.6" width="0.1524" layer="91"/>
-<pinref part="R1" gate="G$1" pin="2"/>
-<wire x1="66.04" y1="35.56" x2="63.5" y2="35.56" width="0.1524" layer="91"/>
-</segment>
-</net>
 <net name="N$7" class="0">
 <segment>
@@
 <wire x1="15.24" y1="27.94" x2="17.78" y2="27.94" width="0.1524" layer="91"/>
 <junction x="17.78" y="27.94"/>
-<label x="17.78" y="33.02" size="1.778" layer="95"/>
+<label x="17.78" y="33.02" size="1.778" layer="95" xref="yes"/>
 </segment>
 <segment>
 <pinref part="U$1" gate="G$1" pin="D6"/>
 <wire x1="111.76" y1="78.74" x2="152.4" y2="78.74" width="0.1524" layer="91"/>
-<label x="152.4" y="78.74" size="1.778" layer="95"/>
+<label x="152.4" y="78.74" size="1.778" layer="95" rot="R270" xref="yes"/>
 </segment>
 </net>
 <net name="N$11" class="0">
 <segment>
-<wire x1="2.54" y1="27.94" x2="0" y2="27.94" width="0.1524" layer="91"/>
 <pinref part="R3" gate="G$1" pin="2"/>
-<wire x1="2.54" y1="27.94" x2="5.08" y2="27.94" width="0.1524" layer="91"/>
-<label x="-2.54" y="27.94" size="1.778" layer="95"/>
+<wire x1="0" y1="27.94" x2="5.08" y2="27.94" width="0.1524" layer="91"/>
+<label x="0" y="30.48" size="1.778" layer="95" rot="R90" xref="yes"/>
+<wire x1="0" y1="27.94" x2="0" y2="30.48" width="0.1524" layer="91"/>
 </segment>
 <segment>
@@
 <wire x1="111.76" y1="68.58" x2="124.46" y2="68.58" width="0.1524" layer="91"/>
 <wire x1="124.46" y1="68.58" x2="124.46" y2="63.5" width="0.1524" layer="91"/>
-<label x="124.46" y="63.5" size="1.778" layer="95"/>
+<label x="124.46" y="63.5" size="1.778" layer="95" xref="yes"/>
 </segment>
 </net>
@@
 </segment>
 </net>
+<net name="N$14" class="0">
+<segment>
+<pinref part="R1" gate="G$1" pin="2"/>
+<wire x1="66.04" y1="35.56" x2="63.5" y2="35.56" width="0.1524" layer="91"/>
+<label x="63.5" y="35.56" size="1.778" layer="95" rot="R90" xref="yes"/>
+</segment>
+<segment>
+<pinref part="U$1" gate="G$1" pin="D12"/>
+<wire x1="119.38" y1="93.98" x2="111.76" y2="93.98" width="0.1524" layer="91"/>
+<label x="119.38" y="96.52" size="1.778" layer="95" xref="yes"/>
+<wire x1="119.38" y1="93.98" x2="119.38" y2="96.52" width="0.1524" layer="91"/>
+</segment>
+</net>

Commit message: schemtic update
Connections:
- net N$8: now also U$1.A6; no longer U$1.A7
Changed lines of the file:
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@@
 <wire x1="78.74" y1="55.88" x2="76.2" y2="55.88" width="0.1524" layer="91"/>
 <junction x="78.74" y="35.56"/>
-<wire x1="76.2" y1="55.88" x2="76.2" y2="68.58" width="0.1524" layer="91"/>
-<pinref part="U$1" gate="G$1" pin="A7"/>
-<wire x1="76.2" y1="68.58" x2="78.74" y2="68.58" width="0.1524" layer="91"/>
+<wire x1="76.2" y1="55.88" x2="76.2" y2="71.12" width="0.1524" layer="91"/>
+<pinref part="U$1" gate="G$1" pin="A6"/>
+<wire x1="78.74" y1="71.12" x2="76.2" y2="71.12" width="0.1524" layer="91"/>
 </segment>
 </net>
